File: Hardware/OrangeHat/2021-07-02 OrangeHat.sch (EAGLE design)
At the start: 57 parts, among them CON1-1 JACK_SMD_3MM5, CON2-1 JACK_SMD_3MM5, IC1-485 SN75176

Commit message: completes initial placement. iterates on routing of power lines.
Parts:
- removed CB1-SRVO1: 1u, 2021-07-02 OrangeHat Library:C-NPOL
- removed CF2-SRVO: 10n, 2021-07-02 OrangeHat Library:C-NPOL
- removed IC-SRVO: ACS712, 2021-07-02 OrangeHat Library:ACS712
- removed MOD-BUCK: 2020-03-18-BUCK, 2021-07-02 OrangeHat Library:2020-03-18-BUCK
- removed RD-485, RU-485: 720, 2021-07-02 OrangeHat Library:R-M2012
- removed RD2-SRVO: 1k, 2021-07-02 OrangeHat Library:R-M2012
- removed RS1-SRVO, RS2-SRVO: 4X 1K, 2021-07-02 OrangeHat Library:RAC164
- removed RT-485: 120, 2021-07-02 OrangeHat Library:R-M2012
- removed RU2-SRVO: 8.2k, 2021-07-02 OrangeHat Library:R-M2012
- removed U$1: SERVO8, 2021-07-02 OrangeHat Library:SERVO8
- added CB-IN-1, CB-RPI-1, CB-SRVO-1, CF-IN-2, CF-RPI-1, CF-SRVO-1: 1u, 2021-07-02 OrangeHat Library:C-NPOL
- added CB-UC-5, CB-UC-6: 100n 50V, 2021-07-02 OrangeHat Library:C-NPOL
- added CF-IN-1, CF-RPI-2, CF-SRVO-2: 10n, 2021-07-02 OrangeHat Library:C-NPOL
- added CON-SRVO: SERVO8-D, 2021-07-02 OrangeHat Library:SERVO8-D
- added CON-UPDI: (no value), 2021-07-02 OrangeHat Library:PINHD-1X3
- added CP-RPI-1: 100uF 6V3, 2021-07-02 OrangeHat Library:C-POLE2.5-5
- added IC-IN-1, IC-RPI-1, IC-SRVO-1: ACS712, 2021-07-02 OrangeHat Library:ACS712
- added LF-UC-2, LF-UC-3: BEAD 500mA, 2021-07-02 OrangeHat Library:L-M2012
- added MOD-PWR: 2020-03-18-BUCK-N5-NHN5, 2021-07-02 OrangeHat Library:2020-03-18-BUCK-N5-NHN5
- added RD-485-1, RU-485-1: 720, 2021-07-02 OrangeHat Library:R0207/2V
- added RD-IN-1, RD-RPI-2, RD-SRVO-2: 1k, 2021-07-02 OrangeHat Library:R-M2012
- added RS-SRVO-2, RS-SRVO-3: 4X 1K, 2021-07-02 OrangeHat Library:RAC164
- added RT-485-1: 120, 2021-07-02 OrangeHat Library:R0207/2V
- added RU-IN-1, RU-RPI-2, RU-SRVO-2: 8.2k, 2021-07-02 OrangeHat Library:R-M2012
- renumbered CB-LCD to CB-LCD-1, CB1-485 to CB-485-2, CB1-SRVO to CB-SRVO-2, CB2-SRVO to CB-SRVO-3, CB3-SRVO to CB-SRVO-4, CF-LCD to CF-LCD-1, CF1-485 to CB-485-1, CON1-1 to CON-485-1, CON2-1 to CON-485-2, CP-SRVO to CP-SRVO-1, CP1-485 to CP-485-1, DL-SRVO to DL-SRVO-1, F-SRVO to F-SRVO-1, IC1-485 to IC-485-1, IMU1 to MOD-IMU-1, LCD16X2 to MOD-LCD-1, LF1-1 to LF-485-1, LF1-SRVO to LF-SRVO-1, LF1-SRVO1 to LF-SRVO-2, LF2-1 to LF-485-2, RD-SRVO to RD-SRVO-1, RD1-LCD to RD-LCD-1, RS1-485 to RS-485-1, RS1-LCD to RS-LCD-1, RS2-485 to RS-485-2, RS2-LCD to RS-LCD-2, RS3-485 to RS-485-3, RS3-SRVO to RS-SRVO-1, RU1-LCD to RU-LCD-1, RU1-SRVO to RU-SRVO-1, RU2-LCD to RU-LCD-2, TP-LCD to TP-LCD-1, TP-SRVO to TP-SRVO-1
Connections:
- net UC-RST renamed RPI-UC-RST
- removed net N$15: CB-SRVO-2.1, LF-SRVO-2.1
- removed net N$3: F-SRVO-1.1
- removed net N$43: IC-UC-1.PD5/AIN5/N1/0-WO5
- removed net VSRVO#A: IC-SRVO.IIN, RU2-SRVO.2, TP-SRVO-1.D
- removed net VSRVO#B: CB-SRVO-2.2, IC-SRVO.IOUT, LF-SRVO-1.1
- new net N$1: CF-RPI-1.2, IC-RPI-1.FILTER
- new net N$2: CF-IN-2.2, IC-IN-1.FILTER
- new net UC-IIN: IC-IN-1.SENSE, IC-UC-1.PD1/AIN1/P3/0-WO1/2-IN1
- new net VIN#: IC-IN-1.IOUT, MOD-PWR.VIN+, RU-IN-1.2
- new net VRPI#A: IC-RPI-1.IIN, MOD-PWR.V5.2A3.0+
- new net VSRVO#A+: IC-SRVO-1.IIN, MOD-PWR.V5.8A3.0+
- new net VSRVO#A-: CB-SRVO-2.1, LF-SRVO-2.1, MOD-PWR.V5.8A3.0-
- new net VSRVO#B+: F-SRVO-1.1, IC-SRVO-1.IOUT, RU-SRVO-2.2
- new net VSRVO#C+: CB-SRVO-2.2, LF-SRVO-1.1, TP-SRVO-1.D
- net CHA485: now also RD-485-1.2, RT-485-1.1; no longer RD-485.2, RT-485.1
- net CHB485: now also RT-485-1.2, RU-485-1.1; no longer RT-485.2, RU-485.1
- net N$19: no longer CB-485-1.1, LF-485-2.1
- net N$20: no longer CB-485-1.2, LF-485-1.1
- net N$21: now also CF-SRVO-1.2, IC-SRVO-1.FILTER; no longer CB1-SRVO1.2, IC-SRVO.FILTER
- net N$23: now also CON-SRVO.8, RS-SRVO-3.4A; no longer RS2-SRVO.1A, U$1.8
- net N$24: now also CON-SRVO.7, RS-SRVO-3.3A; no longer RS2-SRVO.2A, U$1.7
- net N$25: now also CON-SRVO.6, RS-SRVO-3.2A; no longer RS2-SRVO.3A, U$1.6
- net N$26: now also CON-SRVO.5, RS-SRVO-3.1A; no longer RS2-SRVO.4A, U$1.5
- net N$27: now also CON-SRVO.4, RS-SRVO-2.4A; no longer RS1-SRVO.1A, U$1.4
- net N$28: now also CON-SRVO.3, RS-SRVO-2.3A; no longer RS1-SRVO.2A, U$1.3
- net N$29: now also CON-SRVO.2, RS-SRVO-2.2A; no longer RS1-SRVO.3A, U$1.2
- net N$30: now also CON-SRVO.1, RS-SRVO-2.1A; no longer RS1-SRVO.4A, U$1.1
- net UC-IRPI: now also IC-RPI-1.SENSE, IC-UC-1.PD5/AIN5/N1/0-WO5; no longer IC-UC-1.PD2/AIN2/P0/0-WO2/EVOUTD/2-IN2
- net UC-ISRVO: now also IC-SRVO-1.SENSE, IC-UC-1.PD3/AIN3/N0/0-WO3/2-OUT; no longer IC-SRVO.SENSE, IC-UC-1.PD4/AIN4/P1/0-WO4
- net UC-SRVO1: now also RS-SRVO-2.1B; no longer RS1-SRVO.4B
- net UC-SRVO2: now also RS-SRVO-2.2B; no longer RS1-SRVO.3B
- net UC-SRVO3: now also RS-SRVO-2.3B; no longer RS1-SRVO.2B
- net UC-SRVO4: now also RS-SRVO-2.4B; no longer RS1-SRVO.1B
- net UC-SRVO5: now also RS-SRVO-3.1B; no longer RS2-SRVO.4B
- net UC-SRVO6: now also RS-SRVO-3.2B; no longer RS2-SRVO.3B
- net UC-SRVO7: now also RS-SRVO-3.3B; no longer RS2-SRVO.2B
- net UC-SRVO8: now also RS-SRVO-3.4B; no longer RS2-SRVO.1B
- net UC-UPDI: now also CON-UPDI.3
- net UC-VIN: now also CF-IN-1.2, RD-IN-1.2, RU-IN-1.1
- net UC-VRPI: now also CF-RPI-2.2, IC-UC-1.PD4/AIN4/P1/0-WO4, RD-RPI-2.2, RU-RPI-2.1; no longer IC-UC-1.PD1/AIN1/P3/0-WO1/2-IN1
- net UC-VSRVO: now also CF-SRVO-2.2, IC-UC-1.PD2/AIN2/P0/0-WO2/EVOUTD/2-IN2, RD-SRVO-2.2, RU-SRVO-2.1; no longer CF2-SRVO.2, IC-UC-1.PD3/AIN3/N0/0-WO3/2-OUT, RD2-SRVO.2, RU2-SRVO.1
- net V+485: now also RU-485-1.2; no longer RU-485.2
- net V-485: now also RD-485-1.1; no longer RD-485.1
- net VADC+: now also CB-IN-1.2, CB-RPI-1.2, CB-SRVO-1.2, IC-IN-1.+, IC-RPI-1.+, IC-SRVO-1.+
- net VIN+: now also IC-IN-1.IIN; no longer MOD-BUCK.VIN+
- net VIN-: now also MOD-PWR.VIN-; no longer MOD-BUCK.VIN-
- net VRPI+: now also CB-485-1.2, CB-UC-5.2, CP-RPI-1.+, IC-RPI-1.IOUT, LF-485-1.1, LF-UC-2.1, RU-LCD-2.1, RU-RPI-2.2, TP-LCD-1.S; no longer MOD-BUCK.V5.2A3.0+
- net VRPI-: now also CB-485-1.1, CB-UC-5.1, CP-RPI-1.-, LF-485-2.1, LF-UC-3.1, MOD-PWR.V5.2A3.0-; no longer MOD-BUCK.V5.2A3.0-
- net VSRVO+: now also CON-SRVO.+; no longer MOD-BUCK.V5.8A3.0+, U$1.+
- net VSRVO-: now also CON-SRVO.-; no longer MOD-BUCK.V5.8A3.0-, U$1.-
- net VUC+: now also CB-UC-6.2, CON-UPDI.2, LF-UC-2.2; no longer IC-SRVO.+, MOD-BUCK.V5.0A1.0+, RU-LCD-2.1, TP-LCD-1.S
- net VUC-: now also CB-IN-1.1, CB-RPI-1.1, CB-SRVO-1.1, CB-UC-6.1, CF-IN-1.1, CF-IN-2.1, CF-RPI-1.1, CF-RPI-2.1, CF-SRVO-1.1, CF-SRVO-2.1, CON-UPDI.1, IC-IN-1.-, IC-RPI-1.-, IC-SRVO-1.-, LF-UC-3.2, RD-IN-1.1, RD-RPI-2.1, RD-SRVO-2.1; no longer CB1-SRVO1.1, CF2-SRVO.1, IC-SRVO.-, MOD-BUCK.V5.0A1.0-, RD2-SRVO.1
Other:
- note added: "FIXES 2020-03-18 TPS55386 Testing Remove 5.0V1.0A rail Resize 5.8V3.0A rail to 5.2V3.0A rail"
- note added: "POWER"
- note added: "Programmer"
- note removed: "BUCK MODULE"
- moved on the sheet: CB-UC-3, CB-UC-4, CON-PWR, LF-UC-1

Commit message: routing of power lines. complete autoroute of signals.
Parts:
- removed CP-485-1: 100uF 6V3, 2021-07-02 OrangeHat Library:C-POLE2.5-5
- added BTN-UC-1: BTN_NO-M8070, 2021-07-02 OrangeHat Library:BTN_NO-M8070
- added CB-485-3: 1u 50V, 2021-07-02 OrangeHat Library:C-NPOL
- added DL-UC-1, DL-UC-2: LED, 2021-07-02 OrangeHat Library:LED
- added RS-UC-1, RS-UC-2: 330, 2021-07-02 OrangeHat Library:R-M2012
- CB-485-2: value 100n 50V -> 100n 50v
- CB-SRVO-2, CB-SRVO-3: value 1u -> 100n
Connections:
- net N$14 renamed NC-1
- net N$8 renamed NC-2
- removed net N$51: IC-UC-1.PC5/1,RXD/0-WO5
- removed net N$52: IC-UC-1.PC4/1,TXD/0-WO4
- removed net N$62: IC-UC-1.PA6/0,XCK/SCK/0-OUT
- removed net V+485: CB-485-2.2, CP-485-1.+, IC-485-1.V+, LF-485-1.2, RU-485-1.2
- removed net V-485: CB-485-2.1, CP-485-1.-, IC-485-1.V-, LF-485-2.2, RD-485-1.1, RS-485-2.1, RS-485-3.1
- new net N$15: DL-UC-2.+, RS-UC-2.2
- new net N$3: MOD-LCD-1.R/W, RS-LCD-1.3B
- new net N$4: DL-UC-1.+, RS-UC-1.2
- new net UC-BTN-NO: BTN-UC-1.P$2, IC-UC-1.PA6/0,XCK/SCK/0-OUT
- new net UC-LED-1: IC-UC-1.PC4/1,TXD/0-WO4, RS-UC-1.1
- new net UC-LED-2: IC-UC-1.PC5/1,RXD/0-WO5, RS-UC-2.1
- new net V485+: CB-485-2.2, CB-485-3.2, IC-485-1.V+, LF-485-1.2, RU-485-1.2
- new net V485-: CB-485-2.1, CB-485-3.1, IC-485-1.V-, LF-485-2.2, RD-485-1.1, RS-485-2.1, RS-485-3.1
- net VRPI-: now also BTN-UC-1.P$1, CB-LCD-1.1, CF-LCD-1.1, DL-UC-1.-, DL-UC-2.-, MOD-LCD-1.D0, MOD-LCD-1.D1, MOD-LCD-1.D2, MOD-LCD-1.D3, MOD-LCD-1.LIGHT-, MOD-LCD-1.V-, RD-LCD-1.1, RS-LCD-1.3A
- net VUC-: no longer CB-LCD-1.1, CF-LCD-1.1, MOD-LCD-1.D0, MOD-LCD-1.D1, MOD-LCD-1.D2, MOD-LCD-1.D3, MOD-LCD-1.LIGHT-, MOD-LCD-1.R/W, MOD-LCD-1.V-, RD-LCD-1.1
Other:
- note added: "BTN"
- moved on the sheet: CB-485-2, CB-SRVO-2, CB-SRVO-3, CB-SRVO-4, CP-SRVO-1, LF-SRVO-1, LF-SRVO-2

Commit message: completes routing. generates gerber files. validates ERC and DRC with eurocircuit
Parts:
- CB-485-1, CB-485-2: value 100n 50v -> 100n
- CB-485-3: value 1u 50V -> 1u
- CB-IN-1, CB-RPI-1, CB-SRVO-1: value 1u -> 100n
- CB-LCD-1, CB-UC-1, CB-UC-2, CB-UC-3, CB-UC-4, CB-UC-5, CB-UC-6: value 100n 50V -> 100n
- CF-IN-2, CF-RPI-1, CF-SRVO-1: value 1u -> 10n
- CON-UPDI: value (none) -> UPDI
- DL-UC-1: value LED -> GREEN
- DL-UC-2: value LED -> BLUE
- RD-RPI-2, RD-SRVO-2: value 1k -> 10k
- RU-RPI-2, RU-SRVO-2: value 8.2k -> 10k
- TN-UC-1: value MOS-N-SOT23 -> 2N7002
- TP-LCD-1: value MOS-P-SOT23 -> BSS84
- TP-SRVO-1: value MOS-P-TO252 -> 4P03L11
Connections:
- removed net N$17: RS-RPI-1.4A
- removed net N$42: IC-UC-1.PD6/AIN6/P2/2-OUT
- removed net N$49: IC-UC-1.PC7/1,XDIR/EVOUTC
- removed net N$50: IC-UC-1.PC6/1,XCK/1-OUT
- removed net N$53: RS-RPI-1.4B
- removed net NC-1: IC-UC-1.PF4/AIN14/2,TXD/0-WO4/0-WO
- removed net NC-2: IC-UC-1.PF5/AIN15/2,RXD/0-WO5/1-WO
- removed net RPI-SCL: CON-RPI.SCL
- removed net RPI-SDA: CON-RPI.SDA
Other:
- note added: "Discharged 2S - 6.4V Charged 4S - 16.8V"
- note added: "IMU"
- moved on the sheet: BTN-UC-1, CB-485-1, CB-485-2, CB-485-3, CB-IN-1, CB-LCD-1, CB-RPI-1, CB-SRVO-1, CB-SRVO-2, CB-SRVO-3, CB-SRVO-4, CB-UC-1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
